File: tinyprobe2.sch (KiCad schematic (older format))
At the start: 23 parts, among them J1 PRB, J2 USB_B_Micro, J3 DBG, J5 PRGND, J6 LIPO, SW1 BTN, U1 STM32L082KZTx, U2 TP4055, U3 AP7354-33W5-7, U4 ACSA02-41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

Commit message: last rev with the resistors
Parts:
- added J4: EIF, Connector_PinHeader_2.54mm:PinHeader_1x02_P2.54mm_Vertical, symbol Connector_Generic:Conn_01x02
- added J7: VCCOUT, Connector_PinHeader_2.54mm:PinHeader_1x01_P2.54mm_Vertical, symbol Connector_Generic:Conn_01x01
Connections:
- net +3V3: now also J7.1 (Pin_1)
- net ~CHRG: now reaches U1.25 (PA15)
- net ~CHRG: now also U2.1 (~CHRG)
- net EI0: now reaches U1.29 (PB6)
- net EI0: now also J4.1 (Pin_1)
- net EI1: now reaches U1.30 (PB7)
- net EI1: now also J4.2 (Pin_2)
- no-connect marks 12 -> 8
Other:
- moved on the sheet: C1
Changed lines of the file:
@@
 EESchema Schematic File Version 4
+LIBS:tinyprobe2-cache
 EELAYER 26 0
 EELAYER END
@@
 Wire Wire Line
 	7250 1350 6900 1350
-Text Label 1400 4000 0    50   ~ 0
+Text Label 1250 4000 0    50   ~ 0
 VBUS
 Wire Wire Line
-	1650 4000 1550 4000
+	1650 4000 1400 4000
 $Comp
 L Device:R_Small R5
@@
 	2750 4450 2750 4100
 Wire Wire Line
-	2050 4500 1550 4500
+	2050 4500 1400 4500
 Connection ~ 2050 4500
 $Comp
 L Device:C_Small C1
 U 1 1 5BD24FEC
-P 1550 4250
-F 0 "C1" H 1400 4300 50  0000 L CNN
-F 1 "1u" H 1400 4200 50  0000 L CNN
-F 2 "Capacitor_SMD:C_0603_1608Metric_Pad1.05x0.95mm_HandSolder" H 1550 4250 50  0001 C CNN
-F 3 "~" H 1550 4250 50  0001 C CNN
-	1    1550 4250
-	1    0    0    -1
-$EndComp
-Wire Wire Line
-	1550 4150 1550 4000
-Connection ~ 1550 4000
-Wire Wire Line
-	1550 4000 1400 4000
-Wire Wire Line
-	1550 4350 1550 4500
+P 1400 4250
+F 0 "C1" H 1250 4300 50  0000 L CNN
+F 1 "1u" H 1250 4200 50  0000 L CNN
+F 2 "Capacitor_SMD:C_0603_1608Metric_Pad1.05x0.95mm_HandSolder" H 1400 4250 50  0001 C CNN
+F 3 "~" H 1400 4250 50  0001 C CNN
+	1    1400 4250
+	1    0    0    -1
+$EndComp
+Wire Wire Line
+	1400 4150 1400 4000
+Connection ~ 1400 4000
+Wire Wire Line
+	1400 4000 1250 4000
+Wire Wire Line
+	1400 4350 1400 4500
 Text Label 2500 4100 0    50   ~ 0
 PROG
@@
 	6200 1250 6200 1100
 NoConn ~ 4000 1850
-NoConn ~ 5100 2750
 $Comp
 L Connector_Generic:Conn_01x01 J1
@@
 Wire Wire Line
 	1250 1900 1250 2000
-NoConn ~ 1650 4100
 NoConn ~ 8350 3300
 Text Label 5300 1250 2    50   ~ 0
@@
 NoConn ~ 5100 2250
 NoConn ~ 5100 2150
-NoConn ~ 4000 2750
-NoConn ~ 4000 2650
+$Comp
+L Connector_Generic:Conn_01x02 J4
+U 1 1 5BD36A29
+P 1600 2750
+F 0 "J4" H 1520 2425 50  0000 C CNN
+F 1 "EIF" H 1520 2516 50  0000 C CNN
+F 2 "Connector_PinHeader_2.54mm:PinHeader_1x02_P2.54mm_Vertical" H 1600 2750 50  0001 C CNN
+F 3 "~" H 1600 2750 50  0001 C CNN
+	1    1600 2750
+	-1   0    0    1
+$EndComp
+Wire Wire Line
+	1800 2650 2050 2650
+Wire Wire Line
+	1800 2750 2050 2750
+Text Label 2050 2750 2    50   ~ 0
+EI0
+Text Label 2050 2650 2    50   ~ 0
+EI1
+Wire Wire Line
+	4000 2650 3800 2650
+Wire Wire Line
+	4000 2750 3800 2750
+Text Label 3800 2650 0    50   ~ 0
+EI0
+Text Label 3800 2750 0    50   ~ 0
+EI1
+$Comp
+L Connector_Generic:Conn_01x01 J7
+U 1 1 5BD4F46F
+P 1600 3000
+F 0 "J7" H 1520 2775 50  0000 C CNN
+F 1 "VCCOUT" H 1520 2866 50  0000 C CNN
+F 2 "Connector_PinHeader_2.54mm:PinHeader_1x01_P2.54mm_Vertical" H 1600 3000 50  0001 C CNN
+F 3 "~" H 1600 3000 50  0001 C CNN
+	1    1600 3000
+	-1   0    0    1
+$EndComp
+$Comp
+L power:+3V3 #PWR04
+U 1 1 5BD4F690
+P 2000 3000
+F 0 "#PWR04" H 2000 2850 50  0001 C CNN
+F 1 "+3V3" H 2015 3173 50  0000 C CNN
+F 2 "" H 2000 3000 50  0001 C CNN
+F 3 "" H 2000 3000 50  0001 C CNN
+	1    2000 3000
+	0    1    1    0
+$EndComp
+Wire Wire Line
+	2000 3000 1800 3000
+Wire Wire Line
+	1650 4100 1450 4100
+Text Label 1450 4100 0    50   ~ 0
+~CHRG
+Text Label 5500 2750 2    50   ~ 0
+~CHRG
+Wire Wire Line
+	5500 2750 5100 2750
 $EndSCHEMATC

Commit message: days of tuning it
Parts:
- removed RN1, RN2: 49R, Resistor_SMD:R_Array_Concave_4x0603, symbol Device:R_Pack04
- added C4: 100n, Capacitor_SMD:C_0603_1608Metric_Pad1.05x0.95mm_HandSolder, symbol Device:C_Small
- added C5: 1u, Capacitor_SMD:C_0603_1608Metric_Pad1.05x0.95mm_HandSolder, symbol Device:C_Small
- added R10: 33k, Resistor_SMD:R_0603_1608Metric_Pad1.05x0.95mm_HandSolder, symbol Device:R
- added R6, R7, R8: 3k3, Resistor_SMD:R_0603_1608Metric_Pad1.05x0.95mm_HandSolder, symbol Device:R_Small
- added R9: 5, Resistor_SMD:R_0603_1608Metric_Pad1.05x0.95mm_HandSolder, symbol Device:R_Small
- R1: value 220 -> 1k
Connections:
- net DS0 is gone; now on net S3: U1.18 (PA8)
- net DS1 is gone; now on net PROG: U1.15 (PB1)
- net DS3 is gone; now on net S0: U1.13 (PA7)
- net DS4 is gone; now on net S7: U1.12 (PA6)
- net DS5 is gone; now on net S6: U1.11 (PA5)
- net DS6 is gone; now on net S5: U1.10 (PA4)
- net DS7 is gone; now on net S4: U1.9 (PA3)
- net +3V3: now also R9.1; no longer J7.1 (Pin_1)
- net BTN: now also C4.2
- net GND: now also C5.2, R8.1
- net PULL: now also U1.2 (PC14); no longer U1.8 (PA2)
- net S1: now also U1.20 (PA10)
- net S2: now also U1.19 (PA9)
- net VBUS: now also R6.2
- net at D1.1 (K), R1.1: now also R10.2
- net DS2 renamed VBUS_ADC
- net VBUS_ADC: now also R7.2, R8.2
- new net: C4.1, R6.1, R7.1
- new net DSNS: R10.1, U1.8 (PA2)
- new net V3O: C5.1, J7.1 (Pin_1), R9.2
- no-connect marks 8 -> 4
Other:
- note added: "7-segment Displays (Red, Green, Yellow)"
- note added: "Charger & Regulator (Power Supply)"
- note added: "Ext. IF (UART/I2C + 3.3V)"
- note added: "MCU, Button, Debug"
- note added: "Probe"
- note added: "USB (Connector, Attach Wakeup, VBUS Sense)"
- moved on the sheet: C1, C2, C3, D1, J1, J2, J3, J4, J5, J6, J7, R1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
