File: tinyprobe2.kicad_pcb (KiCad board)
At the start: 2 copper layers, 45.1 x 15.2 mm, 23 parts, among them J1 PRB, J2 USB_B_Micro, J3 DBG, J5 PRGND, J6 LIPO, SW1 BTN, U1 STM32L082KZTx, U2 TP4055, U3 AP7354-33W5-7, U4 ACSA02-41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

Commit message: last rev with the resistors
Parts:
- added J4: EIF, Connector_PinHeader_2.54mm:PinHeader_1x02_P2.54mm_Vertical, F.Cu at (79.9, 68.7)
- added J7: VCCOUT, Connector_PinHeader_2.54mm:PinHeader_1x01_P2.54mm_Vertical, F.Cu at (83.6, 65.0)
Connections:
- U1 pad 25: Net-(U1-Pad25) -> /~CHRG
- U1 pad 29: Net-(U1-Pad29) -> /EI0
- U1 pad 30: Net-(U1-Pad30) -> /EI1
- U2 pad 1: Net-(U2-Pad1) -> /~CHRG
Routing:
- net /EI0: track 0.00 -> 30.0 mm, vias 0 -> 2
- net /EI1: track 0.00 -> 27.7 mm, vias 0 -> 2
- net /~CHRG: track 0.00 -> 17.5 mm
- net +3V3: track 52.6 -> 69.6 mm, vias 6 -> 8
- net GND: track 75.3 -> 82.8 mm, vias 3 -> 4
- net /S5: track 38.1 -> 36.6 mm
- net /S6: track 24.9 -> 23.6 mm
- net /S3: track 26.6 -> 25.4 mm
- net /BOOT: track 22.3 -> 23.5 mm
- net /S2: track 25.6 -> 24.4 mm
- net /S1: track 27.1 -> 26.0 mm

Commit message: days of tuning it
Parts:
- removed RN1, RN2: 49R, Resistor_SMD:R_Array_Concave_4x0603
- added C4: 100n, Capacitor_SMD:C_0603_1608Metric_Pad1.05x0.95mm_HandSolder, F.Cu at (109.9, 68.6)
- added C5: 1u, Capacitor_SMD:C_0603_1608Metric_Pad1.05x0.95mm_HandSolder, B.Cu at (83.8, 67.9)
- added R10: 33k, Resistor_SMD:R_0603_1608Metric_Pad1.05x0.95mm_HandSolder, B.Cu at (93.3, 65.4)
- added R6: 3k3, Resistor_SMD:R_0603_1608Metric_Pad1.05x0.95mm_HandSolder, F.Cu at (113.3, 68.6)
- added R7: 3k3, Resistor_SMD:R_0603_1608Metric_Pad1.05x0.95mm_HandSolder, B.Cu at (109.9, 68.6)
- added R8: 3k3, Resistor_SMD:R_0603_1608Metric_Pad1.05x0.95mm_HandSolder, B.Cu at (109.9, 71.8)
- added R9: 5, Resistor_SMD:R_0603_1608Metric_Pad1.05x0.95mm_HandSolder, F.Cu at (84.5, 68.6)
- J2: footprint Connector_USB:USB_Micro-B_GCT_USB3076-30-A -> handy:USB_Micro-B
- R1: value 220 -> 1k
- moved D1 7.24 mm to (90.8, 66.7), turned to 315 degrees
- moved R2 6.82 mm to (87.6, 68.0), turned to 225 degrees
- moved R1 6.79 mm to (87.0, 66.0)
- moved R4 4.96 mm to (90.2, 69.2)
Connections:
- J7 pad 1: +3V3 -> /V3O
- U1 pad 10: /DS6 -> /S5
- U1 pad 11: /DS5 -> /S6
- U1 pad 12: /DS4 -> /S7
- U1 pad 13: /DS3 -> /S0
- U1 pad 14: /DS2 -> /VBUS_ADC
- U1 pad 15: /DS1 -> /PROG
- U1 pad 18: /DS0 -> /S3
- U1 pad 19: Net-(U1-Pad19) -> /S2
- U1 pad 2: Net-(U1-Pad2) -> /PULL
- U1 pad 20: Net-(U1-Pad20) -> /S1
- U1 pad 8: /PULL -> /DSNS
- U1 pad 9: /DS7 -> /S4
Routing:
- net GND: track 82.8 -> 125.9 mm, vias 4 -> 8
- net /PROG: track 2.42 -> 28.4 mm, vias 0 -> 2
- net /VBUS_ADC: track 0.00 -> 14.8 mm
- net +3V3: track 69.6 -> 55.0 mm, vias 8 -> 7
- net /S5: track 36.6 -> 23.4 mm, vias 1 -> 2
- net /S0: track 33.1 -> 43.8 mm
- net /DS3: track 9.13 -> 0.00 mm
- net /PROBE: track 6.31 -> 14.6 mm
- net /DTEST: track 11.5 -> 3.46 mm
- net /DS2: track 7.53 -> 0.00 mm
- net /V3O: track 0.00 -> 6.73 mm
- net /PROBE_3V: track 18.2 -> 11.9 mm
- net /DS1: track 6.11 -> 0.00 mm
- net /S1: track 26.0 -> 31.3 mm, vias 3 -> 2
- net /VBUS: track 42.4 -> 47.0 mm, vias 1 -> 3
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Other:
- board text added: "181031"
- board text added: "TP2"
- board text removed: "181026"

Commit message: add a copying file and idk what else
Routing:
- net /S3: track 27.3 -> 27.9 mm
